File: hardware/proto-v0.1/clock.kicad_sch (KiCad schematic)
At the start: 47 parts, among them J3 BNC REF OUT, J4 BNC 1PPS OUT, J5 BNC AUX OUT, U5 AD5693R, U6 74LVC1G17, U7 74AHCT1G125, U8 74LVC1G125, U9 Si5351C-B-GM, X1 OSC5A2B02, Y1 25MHz

Commit message: Proto-PCB v0.1: placed and routed 4-layer board, PCB generator tools, doc v0.16
Co-Authored-By: Claude Sonnet 5.5 <noreply@anthropic.com>
Claude-Session: https://claude.ai/code/session_01BBEBh5Nhxyv6s49uSZkpLo
Parts:
- X1: footprint Connector_PinHeader_2.54mm:PinHeader_1x05_P2.54mm_Vertical -> HamREF:OCXO_OSC5A2B02_EST

Commit message: Proto-PCB v0.1: fit Fischer AKG 105.26 case (100x80 mm)
Board 100x100 -> 100x80 mm, R1.5 mm corners, no mounting holes (slides into
case grooves), unmasked GND copper strips along both long edges, horizontal
BNC/SMA connectors for the 15.2 mm height budget, router/test-point fixes.
Docs updated to v0.18.

Co-Authored-By: Claude Sonnet 5.5 <noreply@anthropic.com>
Claude-Session: https://claude.ai/code/session_01BBEBh5Nhxyv6s49uSZkpLo
Parts:
- J3, J4, J5: footprint Connector_Coaxial:BNC_Amphenol_031-5539_Vertical -> Connector_Coaxial:BNC_TEConnectivity_1478035_Horizontal; MPN 031-5539 -> 1-1478035-0; Manufacturer Amphenol -> TE Connectivity
