File: hardware/proto-v0.1/gnss.kicad_sch (KiCad schematic)
At the start: 14 parts, among them J2 SMA ANT, U3 LEA-M8S-0, U4 74LVC1G17

Commit message: Proto-PCB v0.1: fit Fischer AKG 105.26 case (100x80 mm)
Board 100x100 -> 100x80 mm, R1.5 mm corners, no mounting holes (slides into
case grooves), unmasked GND copper strips along both long edges, horizontal
BNC/SMA connectors for the 15.2 mm height budget, router/test-point fixes.
Docs updated to v0.18.

Co-Authored-By: Claude Sonnet 5.5 <noreply@anthropic.com>
Claude-Session: https://claude.ai/code/session_01BBEBh5Nhxyv6s49uSZkpLo
Parts:
- J2: footprint Connector_Coaxial:SMA_Amphenol_901-144_Vertical -> Connector_Coaxial:SMA_Amphenol_901-143_Horizontal; MPN 901-144 -> 901-143
Changed lines of the file:
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@@
     (instances
       (project "hamref_proto_v0_1"
-        (path "/9d08a952-c93c-4460-b22e-f5bd0f978dd5/b512301a-c1b3-403a-a35f-8a5c9bc02cc5"
+        (path "/8b52a6c1-3a71-4661-8235-ca3f8f1a695c/4f8b1670-aecc-4869-bfe6-846319b8f146"
           (reference "U3") (unit 1)
         )
@@
       (effects (font (size 1.27 1.27)))
     )
-    (property "Footprint" "Connector_Coaxial:SMA_Amphenol_901-144_Vertical" (at 120 60 0)
+    (property "Footprint" "Connector_Coaxial:SMA_Amphenol_901-143_Horizontal" (at 120 60 0)
       (effects (font (size 1.27 1.27)) hide)
     )
@@
       (effects (font (size 1.27 1.27)) hide)
     )
-    (property "MPN" "901-144" (at 120 60 0)
+    (property "MPN" "901-143" (at 120 60 0)
       (effects (font (size 1.27 1.27)) hide)
     )
@@
     (instances
       (project "hamref_proto_v0_1"
-        (path "/9d08a952-c93c-4460-b22e-f5bd0f978dd5/b512301a-c1b3-403a-a35f-8a5c9bc02cc5"
+        (path "/8b52a6c1-3a71-4661-8235-ca3f8f1a695c/4f8b1670-aecc-4869-bfe6-846319b8f146"
           (reference "J2") (unit 1)
         )
@@
     (instances
       (project "hamref_proto_v0_1"
-        (path "/9d08a952-c93c-4460-b22e-f5bd0f978dd5/b512301a-c1b3-403a-a35f-8a5c9bc02cc5"
+        (path "/8b52a6c1-3a71-4661-8235-ca3f8f1a695c/4f8b1670-aecc-4869-bfe6-846319b8f146"
           (reference "R5") (unit 1)
         )
@@
     (instances
       (project "hamref_proto_v0_1"
-        (path "/9d08a952-c93c-4460-b22e-f5bd0f978dd5/b512301a-c1b3-403a-a35f-8a5c9bc02cc5"
+        (path "/8b52a6c1-3a71-4661-8235-ca3f8f1a695c/4f8b1670-aecc-4869-bfe6-846319b8f146"
           (reference "C12") (unit 1)
         )
@@
     (instances
       (project "hamref_proto_v0_1"
-        (path "/9d08a952-c93c-4460-b22e-f5bd0f978dd5/b512301a-c1b3-403a-a35f-8a5c9bc02cc5"
+        (path "/8b52a6c1-3a71-4661-8235-ca3f8f1a695c/4f8b1670-aecc-4869-bfe6-846319b8f146"
           (reference "C13") (unit 1)
         )
@@
     (instances
       (project "hamref_proto_v0_1"
-        (path "/9d08a952-c93c-4460-b22e-f5bd0f978dd5/b512301a-c1b3-403a-a35f-8a5c9bc02cc5"
+        (path "/8b52a6c1-3a71-4661-8235-ca3f8f1a695c/4f8b1670-aecc-4869-bfe6-846319b8f146"
           (reference "C14") (unit 1)
         )
@@
     (instances
       (project "hamref_proto_v0_1"
-        (path "/9d08a952-c93c-4460-b22e-f5bd0f978dd5/b512301a-c1b3-403a-a35f-8a5c9bc02cc5"
+        (path "/8b52a6c1-3a71-4661-8235-ca3f8f1a695c/4f8b1670-aecc-4869-bfe6-846319b8f146"
           (reference "C15") (unit 1)
         )
@@
     (instances
       (project "hamref_proto_v0_1"
-        (path "/9d08a952-c93c-4460-b22e-f5bd0f978dd5/b512301a-c1b3-403a-a35f-8a5c9bc02cc5"
+        (path "/8b52a6c1-3a71-4661-8235-ca3f8f1a695c/4f8b1670-aecc-4869-bfe6-846319b8f146"
           (reference "C16") (unit 1)
         )
@@
     (instances
       (project "hamref_proto_v0_1"
-        (path "/9d08a952-c93c-4460-b22e-f5bd0f978dd5/b512301a-c1b3-403a-a35f-8a5c9bc02cc5"
+        (path "/8b52a6c1-3a71-4661-8235-ca3f8f1a695c/4f8b1670-aecc-4869-bfe6-846319b8f146"
           (reference "U4") (unit 1)
         )
@@
     (instances
       (project "hamref_proto_v0_1"
-        (path "/9d08a952-c93c-4460-b22e-f5bd0f978dd5/b512301a-c1b3-403a-a35f-8a5c9bc02cc5"
+        (path "/8b52a6c1-3a71-4661-8235-ca3f8f1a695c/4f8b1670-aecc-4869-bfe6-846319b8f146"
           (reference "C17") (unit 1)
         )
@@
     (instances
       (project "hamref_proto_v0_1"
-        (path "/9d08a952-c93c-4460-b22e-f5bd0f978dd5/b512301a-c1b3-403a-a35f-8a5c9bc02cc5"
+        (path "/8b52a6c1-3a71-4661-8235-ca3f8f1a695c/4f8b1670-aecc-4869-bfe6-846319b8f146"
           (reference "TP7") (unit 1)
         )
@@
     (instances
       (project "hamref_proto_v0_1"
-        (path "/9d08a952-c93c-4460-b22e-f5bd0f978dd5/b512301a-c1b3-403a-a35f-8a5c9bc02cc5"
+        (path "/8b52a6c1-3a71-4661-8235-ca3f8f1a695c/4f8b1670-aecc-4869-bfe6-846319b8f146"
           (reference "TP8") (unit 1)
         )
@@
     (instances
       (project "hamref_proto_v0_1"
-        (path "/9d08a952-c93c-4460-b22e-f5bd0f978dd5/b512301a-c1b3-403a-a35f-8a5c9bc02cc5"
+        (path "/8b52a6c1-3a71-4661-8235-ca3f8f1a695c/4f8b1670-aecc-4869-bfe6-846319b8f146"
           (reference "TP9") (unit 1)
         )
@@
     (instances
       (project "hamref_proto_v0_1"
-        (path "/9d08a952-c93c-4460-b22e-f5bd0f978dd5/b512301a-c1b3-403a-a35f-8a5c9bc02cc5"
+        (path "/8b52a6c1-3a71-4661-8235-ca3f8f1a695c/4f8b1670-aecc-4869-bfe6-846319b8f146"
           (reference "R6") (unit 1)
         )
